File: TEST141/TEST141Run2/TEST141/TEST141.kicad_pcb (KiCad board)
At the start: 2 copper layers, 95.8 x 72.3 mm, 160 parts, among them IC1 STM32G030K6T6TR, IC2 W25Q32JVTBIQ, J1 12401610E4_2A, J2 GSB3CN1330DSHR, SW1 TSSF631NJHU

Commit message: Run 2 Ordered
The second run of the test order:
 - changed position of components to fit the EMC disconnect bracket on
 - EMC disconnect added
 - USB-C cell updated
Parts:
- J1: footprint ImportedParts:3432-2001 -> ImportedParts:3432-0901
